Commit message: Added basic boat model with 2 hulls and one beam

File: urdf/foilboat_components.xacro (robot description, xacro)
@@ -1,31 +1,69 @@
 <?xml version="1.0"?>
 <robot name="foilboat" xmlns:xacro="http://www.ros.org/wiki/xacro">
-    <xacro name="hull" params="name port">
-        <link name="${name}_hull">
-            <inertial>
-                <origin xyz="0 0 0" rpy="0 0 0"/>
-                <mass value="${hullMass}"/>
-                <xacro:box_inertia m="${hullMass}" x="${hullX}" y="${hullY}" z="${hullZ}"/>
-            </inertial>
-            <collision>
-                <origin xyz="0 0 0" rpy="0 0 0"/>
-                <geometry>
-                    <box size="${hullX} ${hullY} ${hullZ}"/>
-                </geometry>
-            </collision>
-            <visual>
-                <origin xyz="0 0 0" rpy="0 0 0"/>
-                <geometry>
-                    <box size="${hullX} ${hullY} ${hullZ}"/>
-                </geometry>
-                <!-- Port/Starboard colors -->
-                <xacro:if value="${left == 1}">
-                    <material name="red"/>
-                </xacro:if>
-                <xacro:unless value="${left == 1}">
-                    <material name="green"/>
-                </xacro:unless>
-            </visual>
-        </link>
-    </xacro>
+  <xacro:include filename="$(find foilboat_description)/urdf/macros.xacro" />
+  <xacro:macro name="beam" params="name front">
+    <link name="${name}_beam">
+      <inertia>
+        <origin xyz="0 0 0" rpy="0 0 0"/>
+        <mass value="${beamMass}"/>
+        <xacro:box_inertia m="${beamMass}" x="${beamX}" y="${beamY}" z="${beamZ}"/>
+      </inertia>
+      <collision>
+        <origin xyz="0 0 0" rpy="0 0 0" />
+        <geometry>
+          <box size="${beamX} ${beamY} ${beamZ}" />
+        </geometry>
+      </collision>
+      <visual>
+        <origin xyz="0 0 0" rpy="0 0 0"/>
+        <geometry>
+          <box size="${beamX} ${beamY} ${beamZ}"/>
+        </geometry>
+        <material name="grey"/>
+      </visual>
+    </link>
+    <joint name="${name}_base_joint" type="fixed">
+      <parent link="base_link" />
+      <child link="${name}_beam" />
+      <xacro:if value="${front == 1}">
+        <origin xyz="0 0 0" rpy="0 0 0" />
+      </xacro:if>
+      <xacro:unless value="${front == 1}">
+        <origin xyz="${-hullX + beamX/2} 0 0" rpy="0 0 0" />
+      </xacro:unless>
+    </joint>
+  </xacro:macro>
+  <xacro:macro name="hull" params="name port">
+    <link name="${name}_hull">
+      <inertial>
+        <origin xyz="0 0 0" rpy="0 0 0"/>
+        <mass value="${hullMass}"/>
+        <xacro:box_inertia m="${hullMass}" x="${hullX}" y="${hullY}" z="${hullZ}"/>
+      </inertial>
+      <collision>
+        <origin xyz="0 0 0" rpy="0 0 0"/>
+        <geometry>
+          <box size="${hullX} ${hullY} ${hullZ}"/>
+        </geometry>
+      </collision>
+      <visual>
+        <origin xyz="0 0 0" rpy="0 0 0"/>
+        <geometry>
+          <box size="${hullX} ${hullY} ${hullZ}"/>
+        </geometry>
+        <!-- Port/Starboard colors -->
+        <xacro:if value="${port == 1}">
+          <material name="red"/>
+        </xacro:if>
+        <xacro:unless value="${port == 1}">
+          <material name="green"/>
+        </xacro:unless>
+      </visual>
+    </link>
+    <joint name="${name}_hull_beam_joint" type="fixed">
+      <parent link="front_beam" />
+      <child link="${name}_hull" />
+      <origin xyz="0 ${port * (beamY/2 - hullY/2)} ${-hullZ/2}" rpy="0 0 0" />
+    </joint>
+  </xacro:macro>
 </robot>

File: urdf/foilboat_model.xacro (robot description, xacro)
@@ -1,14 +1,45 @@
 <?xml version="1.0"?>
 <robot name="foilboat" xmlns:xacro="http://www.ros.org/wiki/xacro">
-    <xacro:include filename="$(find foilboat_description)/urdf/materials.xacro" />
-    <xacro:include filename="$(find foilboat_description)/urdf/foilboat_components.xacro" />
-    <xacro:property name="hullLength" value="5.25" />
-    <xacro:property name="hullBeam" value="2.59" />
-    <xacro:property name="hullMass" value="130"/>
-    <xacro:property name="hullX_dim" value="${hullLength}"/>
-    <xacro:property name="hullY_dim" value="0.3"/>
-    <xacro:property name="hullZ_dim" value="0.5" />
-    <xacro:property name="hullX_pos" value="0"/>
-    <xacro:property name="hullY_pos" value="${hullBeam}/2"/>
-    <xacro:property name="hullZ_pos" value="0"/>
+  <xacro:include filename="$(find foilboat_description)/urdf/materials.xacro" />
+  <xacro:include filename="$(find foilboat_description)/urdf/foilboat_components.xacro" />
+  <xacro:include filename="$(find foilboat_description)/urdf/macros.xacro" />
+  <xacro:property name="length" value="5.25" />
+  <xacro:property name="width" value="2.59" />
+  <xacro:property name="hullMass" value="40" />
+  <xacro:property name="hullX" value="${length}" />
+  <xacro:property name="hullY" value="0.3" />
+  <xacro:property name="hullZ" value="0.5" />
+  <xacro:property name="beamMass" value="15" />
+  <xacro:property name="beamX" value="0.2" />
+  <xacro:property name="beamY" value="${width - hullZ}" />
+  <xacro:property name="beamZ" value="0.1" />
+  <link name="base_link" />
+  <xacro:beam name="front" front="1" />
+  <xacro:hull name="left" port="1" />
+  <xacro:hull name="right" port="-1" />
+  <link name="plane_ros::imu_link">
+      <visual>
+          <origin xyz="0 0 0" rpy="0 0 0"/>
+          <geometry>
+              <sphere radius="0.1"/>
+          </geometry>
+          <material name="orange"/>
+      </visual>
+      <collision>
+          <origin xyz="0 0 0" rpy="0 0 0" />
+          <geometry>
+              <sphere radius="0.1" />
+          </geometry>
+      </collision>
+      <inertial>
+          <origin xyz="0 0 0" rpy="0 0 0" />
+          <mass value="1" />
+          <xacro:sphere_inertia m="1" r="0.1" />
+      </inertial>
+  </link>
+  <joint name="plane_ros::imu_link_joint" type="fixed">
+      <parent link="front_beam"/>
+      <child link="plane_ros::imu_link"/>
+      <origin xyz="0 0 0" rpy="${pi} 0 ${pi/2}"/>
+  </joint>
 </robot>

Commit message: Model: Added back beam

File: urdf/foilboat_components.xacro (robot description, xacro)
@@ -30,5 +30,5 @@
       </xacro:if>
       <xacro:unless value="${front == 1}">
-        <origin xyz="${-hullX + beamX/2} 0 0" rpy="0 0 0" />
+        <origin xyz="${-hullX/2 + beamX/2} 0 0" rpy="0 0 0" />
       </xacro:unless>
     </joint>

File: urdf/foilboat_model.xacro (robot description, xacro)
@@ -16,4 +16,5 @@
   <link name="base_link" />
   <xacro:beam name="front" front="1" />
+  <xacro:beam name="back" front="-1"/>
   <xacro:hull name="left" port="1" />
   <xacro:hull name="right" port="-1" />
@@ -41,5 +42,5 @@
     <parent link="front_beam"/>
     <child link="imu_link"/>
-    <origin xyz="0 0 0" rpy="${pi} 0 ${pi/2}"/>
+    <origin xyz="0 0 0" rpy="${pi} 0 0"/>
   </joint>
   <link name="toughsonic_link">
