Commit message: Model: Added rear beam to simulation model

File: urdf/planesim_model.xacro (robot description, xacro)
@@ -16,4 +16,5 @@
   <link name="base_link" />
   <xacro:beam name="front" front="1" />
+  <xacro:beam name="back" front="-1" />
   <xacro:hull name="left" port="1" />
   <xacro:hull name="right" port="-1" />
@@ -41,5 +42,5 @@
       <parent link="front_beam"/>
       <child link="plane_ros::imu_link"/>
-      <origin xyz="0 0 0" rpy="${pi} 0 ${pi/2}"/>
+      <origin xyz="0 0 0" rpy="0 0 0"/>
   </joint>
 </robot>

Commit message: Sim model: Added GPS

File: urdf/planesim_model.xacro (robot description, xacro)
@@ -44,3 +44,28 @@
       <origin xyz="0 0 0" rpy="0 0 0"/>
   </joint>
+  <link name="gps_link">
+    <visual>
+      <origin xyz="0 0 0" rpy="0 0 0"/>
+      <geometry>
+        <sphere radius="0.1"/>
+      </geometry>
+      <material name="orange"/>
+    </visual>
+    <collision>
+      <origin xyz="0 0 0" rpy="0 0 0" />
+      <geometry>
+        <sphere radius="0.1" />
+      </geometry>
+    </collision>
+    <inertial>
+      <origin xyz="0 0 0" rpy="0 0 0" />
+      <mass value="1" />
+      <xacro:sphere_inertia m="1" r="0.1" />
+    </inertial>
+  </link>
+  <joint name="gps_link_joint" type="fixed">
+    <parent link="front_beam"/>
+    <child link="gps_link"/>
+    <origin xyz="0 0 0" rpy="0 0 0"/>
+  </joint>
 </robot>
