Commit message: Real model: Updated link names to reflect real frameID's

File: urdf/foilboat_model.xacro (robot description, xacro)
@@ -18,5 +18,5 @@
   <xacro:hull name="left" port="1" />
   <xacro:hull name="right" port="-1" />
-  <link name="plane_ros::imu_link">
+  <link name="imu_link">
       <visual>
           <origin xyz="0 0 0" rpy="0 0 0"/>
@@ -38,7 +38,7 @@
       </inertial>
   </link>
-  <joint name="plane_ros::imu_link_joint" type="fixed">
+  <joint name="imu_link_joint" type="fixed">
       <parent link="front_beam"/>
-      <child link="plane_ros::imu_link"/>
+      <child link="imu_link"/>
       <origin xyz="0 0 0" rpy="${pi} 0 ${pi/2}"/>
   </joint>

Commit message: Real model: Fixed indentation

File: urdf/foilboat_model.xacro (robot description, xacro)
@@ -19,27 +19,27 @@
   <xacro:hull name="right" port="-1" />
   <link name="imu_link">
-      <visual>
-          <origin xyz="0 0 0" rpy="0 0 0"/>
-          <geometry>
-              <sphere radius="0.1"/>
-          </geometry>
-          <material name="orange"/>
-      </visual>
-      <collision>
-          <origin xyz="0 0 0" rpy="0 0 0" />
-          <geometry>
-              <sphere radius="0.1" />
-          </geometry>
-      </collision>
-      <inertial>
-          <origin xyz="0 0 0" rpy="0 0 0" />
-          <mass value="1" />
-          <xacro:sphere_inertia m="1" r="0.1" />
-      </inertial>
+    <visual>
+      <origin xyz="0 0 0" rpy="0 0 0"/>
+      <geometry>
+        <sphere radius="0.1"/>
+      </geometry>
+      <material name="orange"/>
+    </visual>
+    <collision>
+      <origin xyz="0 0 0" rpy="0 0 0" />
+      <geometry>
+        <sphere radius="0.1" />
+      </geometry>
+    </collision>
+    <inertial>
+      <origin xyz="0 0 0" rpy="0 0 0" />
+      <mass value="1" />
+      <xacro:sphere_inertia m="1" r="0.1" />
+    </inertial>
   </link>
   <joint name="imu_link_joint" type="fixed">
-      <parent link="front_beam"/>
-      <child link="imu_link"/>
-      <origin xyz="0 0 0" rpy="${pi} 0 ${pi/2}"/>
+    <parent link="front_beam"/>
+    <child link="imu_link"/>
+    <origin xyz="0 0 0" rpy="${pi} 0 ${pi/2}"/>
   </joint>
 </robot>

Commit message: Added ultrasonic sensor

File: urdf/foilboat_model.xacro (robot description, xacro)
@@ -43,3 +43,28 @@
     <origin xyz="0 0 0" rpy="${pi} 0 ${pi/2}"/>
   </joint>
+  <link name="toughsonic_link">
+    <visual>
+      <origin xyz="0 0 0" rpy="0 0 0"/>
+      <geometry>
+        <sphere radius="0.1"/>
+      </geometry>
+      <material name="orange"/>
+    </visual>
+    <collision>
+      <origin xyz="0 0 0" rpy="0 0 0" />
+      <geometry>
+        <sphere radius="0.1" />
+      </geometry>
+    </collision>
+    <inertial>
+      <origin xyz="0 0 0" rpy="0 0 0" />
+      <mass value="1" />
+      <xacro:sphere_inertia m="1" r="0.1" />
+    </inertial>
+  </link>
+  <joint name="toughsonic_link_joint" type="fixed">
+    <parent link="front_beam"/>
+    <child link="toughsonic_link"/>
+    <origin xyz="0 0 0" rpy="0 0 0"/>
+  </joint>
 </robot>

Commit message: Foilboat model: Added gps and sensor box

File: urdf/foilboat_model.xacro (robot description, xacro)
@@ -19,29 +19,4 @@
   <xacro:hull name="left" port="1" />
   <xacro:hull name="right" port="-1" />
-  <link name="imu_link">
-    <visual>
-      <origin xyz="0 0 0" rpy="0 0 0"/>
-      <geometry>
-        <sphere radius="0.1"/>
-      </geometry>
-      <material name="orange"/>
-    </visual>
-    <collision>
-      <origin xyz="0 0 0" rpy="0 0 0" />
-      <geometry>
-        <sphere radius="0.1" />
-      </geometry>
-    </collision>
-    <inertial>
-      <origin xyz="0 0 0" rpy="0 0 0" />
-      <mass value="1" />
-      <xacro:sphere_inertia m="1" r="0.1" />
-    </inertial>
-  </link>
-  <joint name="imu_link_joint" type="fixed">
-    <parent link="front_beam"/>
-    <child link="imu_link"/>
-    <origin xyz="0 0 0" rpy="${pi} 0 0"/>
-  </joint>
   <link name="toughsonic_link">
     <visual>
@@ -69,3 +44,79 @@
     <origin xyz="0 0 0" rpy="0 0 0"/>
   </joint>
+  <link name="sensor_box_link">
+    <visual>
+      <origin xyz="0 0 0" rpy="0 0 0"/>
+      <geometry>
+        <sphere radius="0.1"/>
+      </geometry>
+      <material name="black"/>
+    </visual>
+    <collision>
+      <origin xyz="0 0 0" rpy="0 0 0" />
+      <geometry>
+        <sphere radius="0.1" />
+      </geometry>
+    </collision>
+    <inertial>
+      <origin xyz="0 0 0" rpy="0 0 0" />
+      <mass value="1" />
+      <xacro:sphere_inertia m="1" r="0.1" />
+    </inertial>
+  </link>
+  <joint name="sensor_box_link_joint" type="fixed">
+    <parent link="front_beam" />
+    <child link="sensor_box_link" />
+    <origin xyz="0 0 0" rpy="0 0 0" />
+  </joint>
+  <link name="imu_link">
+    <visual>
+      <origin xyz="0 0 0" rpy="0 0 0"/>
+      <geometry>
+        <sphere radius="0.1"/>
+      </geometry>
+      <material name="orange"/>
+    </visual>
+    <collision>
+      <origin xyz="0 0 0" rpy="0 0 0" />
+      <geometry>
+        <sphere radius="0.1" />
+      </geometry>
+    </collision>
+    <inertial>
+      <origin xyz="0 0 0" rpy="0 0 0" />
+      <mass value="1" />
+      <xacro:sphere_inertia m="1" r="0.1" />
+    </inertial>
+  </link>
+  <joint name="imu_link_joint" type="fixed">
+    <parent link="sensor_box_link"/>
+    <child link="imu_link"/>
+    <origin xyz="0 0 0" rpy="${pi} 0 0"/>
+  </joint>
+  <!-- GPS -->
+  <link name="m8u">
+    <visual>
+      <origin xyz="0 0 0" rpy="0 0 0"/>
+      <geometry>
+        <sphere radius="0.1"/>
+      </geometry>
+      <material name="orange"/>
+    </visual>
+    <collision>
+      <origin xyz="0 0 0" rpy="0 0 0" />
+      <geometry>
+        <sphere radius="0.1" />
+      </geometry>
+    </collision>
+    <inertial>
+      <origin xyz="0 0 0" rpy="0 0 0" />
+      <mass value="1" />
+      <xacro:sphere_inertia m="1" r="0.1" />
+    </inertial>
+  </link>
+  <joint name="m8u_joint" type="fixed">
+    <parent link="sensor_box_link"/>
+    <child link="gps_link"/>
+    <origin xyz="0 0 0" rpy="0 0 0"/>
+  </joint>
 </robot>

Commit message: Foilboat model: Fixed gps joint child link name

File: urdf/foilboat_model.xacro (robot description, xacro)
@@ -117,5 +117,5 @@
   <joint name="m8u_joint" type="fixed">
     <parent link="sensor_box_link"/>
-    <child link="gps_link"/>
+    <child link="m8u"/>
     <origin xyz="0 0 0" rpy="0 0 0"/>
   </joint>

Commit message: Foilboat model: Added offset for sensor box

File: urdf/foilboat_model.xacro (robot description, xacro)
@@ -67,5 +67,5 @@
     <parent link="front_beam" />
     <child link="sensor_box_link" />
-    <origin xyz="0 0 0" rpy="0 0 0" />
+    <origin xyz="0 0 0" rpy="0 -0.087 0" />
   </joint>
   <link name="imu_link">
